Commit message: Arm URDF

File: experiment/arm.urdf (robot description, URDF)
Before this commit: robot snapper_mini, 6 links, 5 joints
Links:
- removed link base-link
- removed link trunk
- added link base; visual cylinder length=0.035 radius=0.025
- added link torso; visual cylinder length=0.02 radius=0.01
- link forearm: geometry visual cylinder length=0.05 radius=0.01
- link hand: geometry visual cylinder length=0.07 radius=0.01
- link upper-arm: geometry visual cylinder length=0.05 radius=0.02
Joints:
- removed joint torso
- added joint hip: type continuous, parent base, child torso, origin xyz=0 0 0.035 rpy=0 0 0, axis 0 0 1
- joint base-joint: child base-link -> base
- joint elbow: origin xyz=0 0 0 rpy=0 0 0 -> xyz=0 0.02 0.05 rpy=0 0 0
- joint shoulder: origin xyz=0 0 0 rpy=0 0 0 -> xyz=0 0 0.02 rpy=0 0 0; parent trunk -> torso
- joint wrist: origin xyz=0 0 0 rpy=0 0 0 -> xyz=0 0 0.05 rpy=0 0 0
